File: rancilio-pid/Platinendesign/AIO_PCB/RancilioAIOPID/RancilioAIOPID.sch (KiCad schematic (older format))
At the start: 25 parts, among them J1 Screw_Terminal_Heat, J10 Screw_Terminal_TSIC_Sens, J2 Screw_Terminal_Valve, J3 Screw_Terminal_Pump, J4 Screw_Terminal_220V, J5 Conn_01x15, J5 Screw_Terminal_5V, J6 Conn_01x15, J6 Screw_Terminal_SW_Water, J7 Screw_Terminal_SW_Brew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

Commit message: Doku and PCB
Other:
- note added: "ToDos:\nPull Up /Down Widerstände\nSchaltung Relais\nSchaltung LED Main SW\nTerminal Switch LED"
Changed lines of the file:
@@
 Wire Wire Line
 	5000 2150 3850 2150
+Text Notes 4200 1050 0    50   ~ 0
+ToDos:\nPull Up /Down Widerstände\nSchaltung Relais\nSchaltung LED Main SW\nTerminal Switch LED
 $EndSCHEMATC
