File: doc/Platinendesign/AIO_PCB/RancilioAIOPID/RancilioAIOPID.sch (KiCad schematic (older format))
At the start: 25 parts, among them J1 Screw_Terminal_Heat, J10 Screw_Terminal_TSIC_Sens, J2 Screw_Terminal_Valve, J3 Screw_Terminal_Pump, J4 Screw_Terminal_220V, J5 Conn_01x15, J5 Screw_Terminal_5V, J6 Conn_01x15, J6 Screw_Terminal_SW_Water, J7 Screw_Terminal_SW_Brew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

Commit message: Update Schema
Parts:
- added D1: 1N4148, Diode_THT:D_DO-35_SOD27_P7.62mm_Horizontal, symbol Diode:1N4148
- added J11: Screw_Terminal_Main_LED, symbol Connector:Screw_Terminal_01x02
- added Q1: BC337, Package_TO_SOT_THT:TO-92_Inline, symbol Transistor_BJT:BC337
- added R10, R11, R9: 75R, symbol Device:R
- added R7: 270R, symbol Device:R
- added R8: 150R, symbol Device:R
- K1: value FINDER-40.52 -> FINDER-40.52.7
- gave numbers to parts that had none: 2
Connections:
- net at J5.2 (Pin_2), U1.2, U2.2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: now also J10.3 (Pin_3), J5.2 (Pin_2), J6.14 (Pin_14), J6.2 (Pin_2), J7.2 (Pin_2), J8.2 (Pin_2), Q1.3 (E)
- net at K1.A1: now also J10.1 (Pin_1), J5.1 (Pin_1), J6.15 (Pin_15), D1.1 (K), R10.1, R11.2, R8.1, R9.1
- net at K1.A2: now also D1.2 (A), J11.2 (Pin_2), Q1.1 (C)
- net at J5.4 (Pin_4): now also R7.2
- new net: J8.1 (Pin_1), R11.1
- new net: J7.1 (Pin_1), R10.2
- new net: J6.1 (Pin_1), R9.2
- new net: Q1.2 (B), R7.1
- new net: J11.1 (Pin_1), R8.2
Other:
- note removed: "ToDos:\nPull Up /Down Widerstände\nSchaltung Relais\nSchaltung LED Main SW\nTerminal Switch LED"
- moved on the sheet: J1, J10, J2, J3, J4, J5, J6, J7, J8, J9, K1, Q1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
